File: schematic-v4/pollbox.sch (KiCad schematic (older format))
At the start: 20 parts, among them P1 CONN_01X15, P10 CONN_01X04, P2 CONN_02X03, P20 CONN_01X04, P3 CONN_01X15, P30 CONN_01X04, P40 CONN_01X04, P50 CONN_01X04, U1 NodeMCU, U2 ULN2803

Commit message: o Filling zones. o Adding drill holes.
Parts:
- added W1, W2, W3, W4: TEST_1P, Connect:1pin, symbol TEST_1P
Other:
- note added: "Mounting holes"
Changed lines of the file:
@@
 $EndDescr
 $Comp
-L GND #PWR01
+L GND #PWR25
 U 1 1 565CA52E
 P 2350 6750
-F 0 "#PWR01" H 2350 6500 50  0001 C CNN
+F 0 "#PWR25" H 2350 6500 50  0001 C CNN
 F 1 "GND" H 2350 6600 50  0000 C CNN
 F 2 "" H 2350 6750 60  0000 C CNN
@@
 $EndComp
 $Comp
-L GND #PWR02
+L GND #PWR24
 U 1 1 565CA58B
 P 4200 6300
-F 0 "#PWR02" H 4200 6050 50  0001 C CNN
+F 0 "#PWR24" H 4200 6050 50  0001 C CNN
 F 1 "GND" H 4200 6150 50  0000 C CNN
 F 2 "" H 4200 6300 60  0000 C CNN
@@
 $EndComp
 $Comp
-L +5V #PWR03
+L +5V #PWR20
 U 1 1 565CB234
 P 2100 4450
-F 0 "#PWR03" H 2100 4300 50  0001 C CNN
+F 0 "#PWR20" H 2100 4300 50  0001 C CNN
 F 1 "+5V" H 2100 4590 50  0000 C CNN
 F 2 "" H 2100 4450 60  0000 C CNN
@@
 $EndComp
 $Comp
-L +5V #PWR04
+L +5V #PWR2
 U 1 1 565CB305
 P 2550 1200
-F 0 "#PWR04" H 2550 1050 50  0001 C CNN
+F 0 "#PWR2" H 2550 1050 50  0001 C CNN
 F 1 "+5V" H 2550 1340 50  0000 C CNN
 F 2 "" H 2550 1200 60  0000 C CNN
@@
 $EndComp
 $Comp
-L +3V3 #PWR05
+L +3V3 #PWR1
 U 1 1 565CB44C
 P 2350 1200
-F 0 "#PWR05" H 2350 1050 50  0001 C CNN
+F 0 "#PWR1" H 2350 1050 50  0001 C CNN
 F 1 "+3V3" H 2350 1340 50  0000 C CNN
 F 2 "" H 2350 1200 60  0000 C CNN
@@
 $EndComp
 $Comp
-L GND #PWR06
+L GND #PWR11
 U 1 1 565CB544
 P 2350 2400
-F 0 "#PWR06" H 2350 2150 50  0001 C CNN
+F 0 "#PWR11" H 2350 2150 50  0001 C CNN
 F 1 "GND" H 2350 2250 50  0000 C CNN
 F 2 "" H 2350 2400 60  0000 C CNN
@@
 $EndComp
 $Comp
-L +3V3 #PWR07
+L +3V3 #PWR21
 U 1 1 56A3DCCD
 P 4100 4450
-F 0 "#PWR07" H 4100 4300 50  0001 C CNN
+F 0 "#PWR21" H 4100 4300 50  0001 C CNN
 F 1 "+3V3" H 4100 4590 50  0000 C CNN
 F 2 "" H 4100 4450 60  0000 C CNN
@@
 SWITCH_1
 $Comp
-L GND #PWR08
+L GND #PWR23
 U 1 1 56A487F8
 P 8400 4850
-F 0 "#PWR08" H 8400 4600 50  0001 C CNN
+F 0 "#PWR23" H 8400 4600 50  0001 C CNN
 F 1 "GND" H 8400 4700 50  0000 C CNN
 F 2 "" H 8400 4850 60  0000 C CNN
@@
 $EndComp
 $Comp
-L +3V3 #PWR09
+L +3V3 #PWR19
 U 1 1 56A48B7F
 P 8600 4300
-F 0 "#PWR09" H 8600 4150 50  0001 C CNN
+F 0 "#PWR19" H 8600 4150 50  0001 C CNN
 F 1 "+3V3" H 8600 4440 50  0000 C CNN
 F 2 "" H 8600 4300 60  0000 C CNN
@@
 $EndComp
 $Comp
-L +5V #PWR010
+L +5V #PWR18
 U 1 1 56A48BC9
 P 8400 4300
-F 0 "#PWR010" H 8400 4150 50  0001 C CNN
+F 0 "#PWR18" H 8400 4150 50  0001 C CNN
 F 1 "+5V" H 8400 4440 50  0000 C CNN
 F 2 "" H 8400 4300 60  0000 C CNN
@@
 $EndComp
 $Comp
-L GND #PWR011
+L GND #PWR22
 U 1 1 56A493D7
 P 7700 4850
-F 0 "#PWR011" H 7700 4600 50  0001 C CNN
+F 0 "#PWR22" H 7700 4600 50  0001 C CNN
 F 1 "GND" H 7700 4700 50  0000 C CNN
 F 2 "" H 7700 4850 60  0000 C CNN
@@
 $EndComp
 $Comp
-L +5V #PWR012
+L +5V #PWR17
 U 1 1 56A4975F
 P 7700 4300
-F 0 "#PWR012" H 7700 4150 50  0001 C CNN
+F 0 "#PWR17" H 7700 4150 50  0001 C CNN
 F 1 "+5V" H 7700 4440 50  0000 C CNN
 F 2 "" H 7700 4300 60  0000 C CNN
@@
 $EndComp
 $Comp
-L +3V3 #PWR013
+L +3V3 #PWR16
 U 1 1 56A497A9
 P 7500 4300
-F 0 "#PWR013" H 7500 4150 50  0001 C CNN
+F 0 "#PWR16" H 7500 4150 50  0001 C CNN
 F 1 "+3V3" H 7500 4440 50  0000 C CNN
 F 2 "" H 7500 4300 60  0000 C CNN
@@
 LED_1
 $Comp
-L +5V #PWR014
+L +5V #PWR4
 U 1 1 573F7C58
 P 4000 1200
-F 0 "#PWR014" H 4000 1050 50  0001 C CNN
+F 0 "#PWR4" H 4000 1050 50  0001 C CNN
 F 1 "+5V" H 4000 1340 50  0000 C CNN
 F 2 "" H 4000 1200 60  0000 C CNN
@@
 $EndComp
 $Comp
-L +3V3 #PWR015
+L +3V3 #PWR3
 U 1 1 573F7C5E
 P 3800 1200
-F 0 "#PWR015" H 3800 1050 50  0001 C CNN
+F 0 "#PWR3" H 3800 1050 50  0001 C CNN
 F 1 "+3V3" H 3800 1340 50  0000 C CNN
 F 2 "" H 3800 1200 60  0000 C CNN
@@
 $EndComp
 $Comp
-L GND #PWR016
+L GND #PWR12
 U 1 1 573F7C64
 P 3800 2400
-F 0 "#PWR016" H 3800 2150 50  0001 C CNN
+F 0 "#PWR12" H 3800 2150 50  0001 C CNN
 F 1 "GND" H 3800 2250 50  0000 C CNN
 F 2 "" H 3800 2400 60  0000 C CNN
@@
 LED_2
 $Comp
-L +5V #PWR017
+L +5V #PWR6
 U 1 1 573F7D0F
 P 5450 1200
-F 0 "#PWR017" H 5450 1050 50  0001 C CNN
+F 0 "#PWR6" H 5450 1050 50  0001 C CNN
 F 1 "+5V" H 5450 1340 50  0000 C CNN
 F 2 "" H 5450 1200 60  0000 C CNN
@@
 $EndComp
 $Comp
-L +3V3 #PWR018
+L +3V3 #PWR5
 U 1 1 573F7D15
 P 5250 1200
-F 0 "#PWR018" H 5250 1050 50  0001 C CNN
+F 0 "#PWR5" H 5250 1050 50  0001 C CNN
 F 1 "+3V3" H 5250 1340 50  0000 C CNN
 F 2 "" H 5250 1200 60  0000 C CNN
@@
 $EndComp
 $Comp
-L GND #PWR019
+L GND #PWR13
 U 1 1 573F7D1B
 P 5250 2400
-F 0 "#PWR019" H 5250 2150 50  0001 C CNN
+F 0 "#PWR13" H 5250 2150 50  0001 C CNN
 F 1 "GND" H 5250 2250 50  0000 C CNN
 F 2 "" H 5250 2400 60  0000 C CNN
@@
 LED_3
 $Comp
-L +5V #PWR020
+L +5V #PWR8
 U 1 1 573F854E
 P 6900 1200
-F 0 "#PWR020" H 6900 1050 50  0001 C CNN
+F 0 "#PWR8" H 6900 1050 50  0001 C CNN
 F 1 "+5V" H 6900 1340 50  0000 C CNN
 F 2 "" H 6900 1200 60  0000 C CNN
@@
 $EndComp
 $Comp
-L +3V3 #PWR021
+L +3V3 #PWR7
 U 1 1 573F8554
 P 6700 1200
-F 0 "#PWR021" H 6700 1050 50  0001 C CNN
+F 0 "#PWR7" H 6700 1050 50  0001 C CNN
 F 1 "+3V3" H 6700 1340 50  0000 C CNN
 F 2 "" H 6700 1200 60  0000 C CNN
@@
 $EndComp
 $Comp
-L GND #PWR022
+L GND #PWR14
 U 1 1 573F855A
 P 6700 2400
-F 0 "#PWR022" H 6700 2150 50  0001 C CNN
+F 0 "#PWR14" H 6700 2150 50  0001 C CNN
 F 1 "GND" H 6700 2250 50  0000 C CNN
 F 2 "" H 6700 2400 60  0000 C CNN
@@
 LED_4
 $Comp
-L +5V #PWR023
+L +5V #PWR10
 U 1 1 573F887E
 P 8350 1200
-F 0 "#PWR023" H 8350 1050 50  0001 C CNN
+F 0 "#PWR10" H 8350 1050 50  0001 C CNN
 F 1 "+5V" H 8350 1340 50  0000 C CNN
 F 2 "" H 8350 1200 60  0000 C CNN
@@
 $EndComp
 $Comp
-L +3V3 #PWR024
+L +3V3 #PWR9
 U 1 1 573F8884
 P 8150 1200
-F 0 "#PWR024" H 8150 1050 50  0001 C CNN
+F 0 "#PWR9" H 8150 1050 50  0001 C CNN
 F 1 "+3V3" H 8150 1340 50  0000 C CNN
 F 2 "" H 8150 1200 60  0000 C CNN
@@
 $EndComp
 $Comp
-L GND #PWR025
+L GND #PWR15
 U 1 1 573F888A
 P 8150 2400
-F 0 "#PWR025" H 8150 2150 50  0001 C CNN
+F 0 "#PWR15" H 8150 2150 50  0001 C CNN
 F 1 "GND" H 8150 2250 50  0000 C CNN
 F 2 "" H 8150 2400 60  0000 C CNN
@@
 Wire Wire Line
 	6450 3150 6000 3150
+$Comp
+L TEST_1P W1
+U 1 1 57A37AA1
+P 8600 5800
+F 0 "W1" H 8600 6070 50  0000 C CNN
+F 1 "TEST_1P" H 8600 6000 50  0000 C CNN
+F 2 "Connect:1pin" H 8800 5800 50  0001 C CNN
+F 3 "" H 8800 5800 50  0000 C CNN
+	1    8600 5800
+	1    0    0    -1
+$EndComp
+$Comp
+L TEST_1P W2
+U 1 1 57A37AFE
+P 8950 5800
+F 0 "W2" H 8950 6070 50  0000 C CNN
+F 1 "TEST_1P" H 8950 6000 50  0000 C CNN
+F 2 "Connect:1pin" H 9150 5800 50  0001 C CNN
+F 3 "" H 9150 5800 50  0000 C CNN
+	1    8950 5800
+	1    0    0    -1
+$EndComp
+$Comp
+L TEST_1P W3
+U 1 1 57A37B3F
+P 9300 5800
+F 0 "W3" H 9300 6070 50  0000 C CNN
+F 1 "TEST_1P" H 9300 6000 50  0000 C CNN
+F 2 "Connect:1pin" H 9500 5800 50  0001 C CNN
+F 3 "" H 9500 5800 50  0000 C CNN
+	1    9300 5800
+	1    0    0    -1
+$EndComp
+Text Notes 8750 6050 0    60   ~ 0
+Mounting holes
+$Comp
+L TEST_1P W4
+U 1 1 57A38328
+P 9650 5800
+F 0 "W4" H 9650 6070 50  0000 C CNN
+F 1 "TEST_1P" H 9650 6000 50  0000 C CNN
+F 2 "Connect:1pin" H 9850 5800 50  0001 C CNN
+F 3 "" H 9850 5800 50  0000 C CNN
+	1    9650 5800
+	1    0    0    -1
+$EndComp
 $EndSCHEMATC

Commit message: o Adding build setup to use kicad-utils to generate schematic-v4.h from the KiCAD schematic.
Connections:
- net labels added: LED_1_OUT, LED_2_OUT, LED_3_OUT, LED_4_OUT, LED_5_OUT
Changed lines of the file:
@@
 LIBS:valves
 LIBS:pollbox
-LIBS:pollbox-cache
 EELAYER 25 0
 EELAYER END
@@
 $EndComp
 Text Label 3100 1950 0    60   ~ 0
-LED_1
+LED_1_OUT
 $Comp
 L +5V #PWR4
@@
 $EndComp
 Text Label 4550 1950 0    60   ~ 0
-LED_2
+LED_2_OUT
 $Comp
 L +5V #PWR6
@@
 $EndComp
 Text Label 6000 1950 0    60   ~ 0
-LED_3
+LED_3_OUT
 $Comp
 L +5V #PWR8
@@
 $EndComp
 Text Label 7450 1950 0    60   ~ 0
-LED_4
+LED_4_OUT
 $Comp
 L +5V #PWR10
@@
 $EndComp
 Text Label 8900 1950 0    60   ~ 0
-LED_5
+LED_5_OUT
 $Comp
 L ULN2803 U2
@@
 	1    0    0    -1
 $EndComp
+Text Label 4950 4800 0    60   ~ 0
+LED_1
+Text Label 4950 5000 0    60   ~ 0
+LED_2
+Text Label 4950 5100 0    60   ~ 0
+LED_3
+Text Label 4950 5400 0    60   ~ 0
+LED_4
+Text Label 4950 5600 0    60   ~ 0
+LED_5
 $EndSCHEMATC
