File: schematic-v5/pollbox.kicad_pcb (KiCad board)
At the start: 2 copper layers, 49.5 x 72.4 mm, 24 parts, among them P1 CONN_01X15, P10 CONN_01X04, P2 CONN_02X03, P20 CONN_01X04, P3 CONN_01X15, P30 CONN_01X04, P40 CONN_01X04, P50 CONN_01X04, U1 NodeMCU_1.0, U2 ULN2803

Commit message: fixed slik screen stuff
Parts:
- HOLE1: value MountingHole_3.2mm_M3 -> M1
- HOLE2: value MountingHole_3.2mm_M3 -> M2
- HOLE3: value MountingHole_3.2mm_M3 -> M4
- HOLE4: value MountingHole_3.2mm_M3 -> M3
- P1, P3: value CONN_01X15 -> (none)
- P10: value CONN_01X04 -> SW_1
- P2: value CONN_02X03 -> Power
- P20: value CONN_01X04 -> SW_2
- P30: value CONN_01X04 -> SW_3
- P40: value CONN_01X04 -> SW_4
- P50: value CONN_01X04 -> SW_5
Other:
- board text added: "5V 3.3V GND"
Changed lines of the file:
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@@
     (area 65.810001 40.48 132.801143 121.927333)
     (thickness 1.6)
-    (drawings 9)
+    (drawings 10)
     (tracks 281)
     (zones 0)
@@
     (34 B.Paste user)
     (35 F.Paste user)
-    (36 B.SilkS user hide)
-    (37 F.SilkS user hide)
+    (36 B.SilkS user)
+    (37 F.SilkS user)
     (38 B.Mask user)
     (39 F.Mask user)
@@
     (aux_axis_origin 77.47 118.745)
     (grid_origin 77.47 119.38)
-    (visible_elements FFFCFF7F)
+    (visible_elements FFFDFF7F)
     (pcbplotparams
       (layerselection 0x3ffff_80000001)
@@
       (padsonsilk false)
       (subtractmaskfromsilk false)
-      (outputformat 4)
+      (outputformat 1)
       (mirror false)
       (drillshape 0)
       (scaleselection 1)
-      (outputdirectory pdf-real))
+      (outputdirectory gerber/))
   )
   (net 0 "")
@@
       (effects (font (size 1 1) (thickness 0.15)))
     )
-    (fp_text value MountingHole_3.2mm_M3 (at 0 4.2) (layer F.Fab)
+    (fp_text value M3 (at 3.81 -3.048) (layer F.Fab)
       (effects (font (size 1 1) (thickness 0.15)))
     )
@@
       (effects (font (size 1 1) (thickness 0.15)))
     )
-    (fp_text value MountingHole_3.2mm_M3 (at 0 4.2) (layer F.Fab)
+    (fp_text value M4 (at -3.937 -2.921) (layer F.Fab)
       (effects (font (size 1 1) (thickness 0.15)))
     )
@@
       (effects (font (size 1 1) (thickness 0.15)))
     )
-    (fp_text value MountingHole_3.2mm_M3 (at 0 4.2) (layer F.Fab)
+    (fp_text value M2 (at -3.302 -3.556) (layer F.Fab)
       (effects (font (size 1 1) (thickness 0.15)))
     )
@@
       (effects (font (size 1 1) (thickness 0.15)))
     )
-    (fp_text value CONN_01X04 (at 0 -3.1) (layer F.Fab)
+    (fp_text value SW_4 (at 0 11.176 90) (layer F.Fab)
       (effects (font (size 1 1) (thickness 0.15)))
     )
@@
       (effects (font (size 1 1) (thickness 0.15)))
     )
-    (fp_text value 100n (at 1.25 2.5 270) (layer F.Fab)
+    (fp_text value 100n (at 5.715 0.127 270) (layer F.Fab)
       (effects (font (size 1 1) (thickness 0.15)))
     )
@@
       (effects (font (size 1 1) (thickness 0.15)))
     )
-    (fp_text value 10k (at 3.81 3.81 90) (layer F.Fab)
+    (fp_text value 10k (at 2.159 -2.159 90) (layer F.Fab)
       (effects (font (size 1 1) (thickness 0.15)))
     )
@@
       (effects (font (size 1 1) (thickness 0.15)))
     )
-    (fp_text value 100n (at 1.25 2.5 270) (layer F.Fab)
+    (fp_text value 100n (at 5.715 0.254 270) (layer F.Fab)
       (effects (font (size 1 1) (thickness 0.15)))
     )
@@
       (effects (font (size 1 1) (thickness 0.15)))
     )
-    (fp_text value 10k (at 3.81 3.81 90) (layer F.Fab)
+    (fp_text value 10k (at 2.159 -2.159 90) (layer F.Fab)
       (effects (font (size 1 1) (thickness 0.15)))
     )
@@
       (effects (font (size 1 1) (thickness 0.15)))
     )
-    (fp_text value 100n (at 1.25 2.5 270) (layer F.Fab)
+    (fp_text value 100n (at 5.715 0.127 270) (layer F.Fab)
       (effects (font (size 1 1) (thickness 0.15)))
     )
@@
       (effects (font (size 1 1) (thickness 0.15)))
     )
-    (fp_text value 100n (at 1.25 2.5 270) (layer F.Fab)
+    (fp_text value 100n (at 5.842 0.127 270) (layer F.Fab)
       (effects (font (size 1 1) (thickness 0.15)))
     )
@@
       (effects (font (size 1 1) (thickness 0.15)))
     )
-    (fp_text value 100n (at 1.25 2.5 270) (layer F.Fab)
+    (fp_text value 100n (at 5.715 0 270) (layer F.Fab)
       (effects (font (size 1 1) (thickness 0.15)))
     )
@@
       (effects (font (size 1 1) (thickness 0.15)))
     )
-    (fp_text value CONN_02X03 (at 0 -3.1) (layer F.Fab)
+    (fp_text value Power (at 0 -3.1) (layer F.Fab)
       (effects (font (size 1 1) (thickness 0.15)))
     )
@@
       (effects (font (size 1 1) (thickness 0.15)))
     )
-    (fp_text value CONN_01X04 (at 0 -3.1) (layer F.Fab)
+    (fp_text value SW_1 (at -0.254 11.303 90) (layer F.Fab)
       (effects (font (size 1 1) (thickness 0.15)))
     )
@@
       (effects (font (size 1 1) (thickness 0.15)))
     )
-    (fp_text value CONN_01X04 (at 0 -3.1) (layer F.Fab)
+    (fp_text value SW_2 (at -0.254 11.684 90) (layer F.Fab)
       (effects (font (size 1 1) (thickness 0.15)))
     )
@@
       (effects (font (size 1 1) (thickness 0.15)))
     )
-    (fp_text value CONN_01X04 (at 0 -3.1) (layer F.Fab)
+    (fp_text value SW_3 (at -0.127 11.43 90) (layer F.Fab)
       (effects (font (size 1 1) (thickness 0.15)))
     )
@@
       (effects (font (size 1 1) (thickness 0.15)))
     )
-    (fp_text value CONN_01X04 (at 0 -3.1) (layer F.Fab)
+    (fp_text value SW_5 (at -0.127 11.43 90) (layer F.Fab)
       (effects (font (size 1 1) (thickness 0.15)))
     )
@@
       (effects (font (size 1 1) (thickness 0.15)))
     )
-    (fp_text value 10k (at 3.81 3.81 90) (layer F.Fab)
+    (fp_text value 10k (at 2.032 -2.159 90) (layer F.Fab)
       (effects (font (size 1 1) (thickness 0.15)))
     )
@@
       (effects (font (size 1 1) (thickness 0.15)))
     )
-    (fp_text value 10k (at 3.81 3.81 90) (layer F.Fab)
+    (fp_text value 10k (at 2.413 -2.159 90) (layer F.Fab)
       (effects (font (size 1 1) (thickness 0.15)))
     )
@@
       (effects (font (size 1 1) (thickness 0.15)))
     )
-    (fp_text value 10k (at 3.81 3.81 90) (layer F.Fab)
+    (fp_text value 10k (at 2.413 -2.159 90) (layer F.Fab)
       (effects (font (size 1 1) (thickness 0.15)))
     )
@@
       (effects (font (size 1 1) (thickness 0.15)))
     )
-    (fp_text value MountingHole_3.2mm_M3 (at 0 4.2) (layer F.Fab)
+    (fp_text value M1 (at 3.556 -3.683) (layer F.Fab)
       (effects (font (size 1 1) (thickness 0.15)))
     )
@@
       (effects (font (size 1 1) (thickness 0.15)))
     )
-    (fp_text value CONN_01X15 (at 0 -3.1 270) (layer F.Fab)
+    (fp_text value "" (at 0 -3.1 270) (layer F.Fab)
       (effects (font (size 1 1) (thickness 0.15)))
     )
@@
       (effects (font (size 1 1) (thickness 0.15)))
     )
-    (fp_text value CONN_01X15 (at 0 -3.1 270) (layer F.Fab)
+    (fp_text value "" (at 0 -3.1 270) (layer F.Fab)
       (effects (font (size 1 1) (thickness 0.15)))
     )
@@
       (effects (font (size 0.889 0.889) (thickness 0.3048)))
     )
-    (fp_text value NodeMCU_1.0 (at 0 0 270) (layer F.SilkS)
-      (effects (font (size 0.889 0.889) (thickness 0.3048)))
+    (fp_text value NodeMCU_1.0 (at 0 0 90) (layer F.Fab)
+      (effects (font (size 1 1) (thickness 0.15)))
     )
     (pad 1 thru_hole oval (at 17.78 11.43) (size 1.7272 2.3) (drill 0.762) (layers *.Cu *.Mask F.SilkS)
@@
       (net 1 +3V3))
   )
+  (gr_text "5V\n\n3.3V\n\nGND" (at 122.047 78.867) (layer F.Fab)
+    (effects (font (size 1 1) (thickness 0.15)) (justify left))
+  )
   (dimension 49.53 (width 0.3) (layer Cmts.User)
